File: pixhawk.sch (EAGLE design)
At the start: 9 parts, among them J201 80-PIN-CARD-EDGE

Commit message: Start pixhawk board redesign
Parts:
- removed JP107: CAN, auv:DF13-4P-1.25DSA
- removed U$2: ILLINOISAUV, auv:ILLINOISAUV
- JP102, JP103, JP104: device auv:DF13-6P-1.25DSA -> auv:PINHD-1X6
- JP105: value POWER -> PWR; device auv:DF13-6P-1.25DSA -> auv:PINHD-1X6
- JP106: device auv:DF13-4P-1.25DSA -> auv:PINHD-1X4
Connections:
- net CAN_H: no longer JP107.2
- net CAN_L: no longer JP107.3
- net GND: no longer JP107.4
