File: cardedge_connector_breakout.brd (EAGLE design)
At the start: 111.7 x 44.1 mm, 3 parts

Commit message: Updates and fixes
Parts:
- removed U$2: ILLINOISAUV, auv:ILLINOISAUV
- moved JP1 21.6 mm to (55.9, 19.1)
Routing:
- net N$6: track 36.9 -> 15.1 mm
- net N$33: track 36.9 -> 15.1 mm
- net N$24: track 36.9 -> 15.1 mm
- net N$15: track 36.9 -> 15.1 mm
- net N$34: track 36.9 -> 15.1 mm
- net N$25: track 36.9 -> 15.1 mm
- net N$16: track 36.9 -> 15.1 mm
- net N$7: track 36.9 -> 15.1 mm
- net N$35: track 36.8 -> 15.1 mm
- net N$26: track 36.8 -> 15.1 mm
- net N$8: track 36.8 -> 15.1 mm
- net N$17: track 36.8 -> 15.1 mm
- net N$9: track 36.8 -> 15.1 mm
- net N$36: track 36.8 -> 15.1 mm
- net N$27: track 36.8 -> 15.1 mm
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Other:
- board size 111.7 x 44.1 mm -> 111.7 x 22.5 mm
