File: cardedge_connector_breakout.sch (EAGLE design)
At the start: 3 parts

Commit message: Updates and fixes
Parts:
- removed U$2: ILLINOISAUV, auv:ILLINOISAUV
Changed lines of the file:
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@@
 <?xml version="1.0" encoding="utf-8"?>
 <!DOCTYPE eagle SYSTEM "eagle.dtd">
-<eagle version="8.4.0">
+<eagle version="8.6.0">
 <drawing>
 <settings>
@@
 <part name="U$1" library="auv" deviceset="TE-2-5530843-0" device=""/>
 <part name="JP1" library="auv" deviceset="PINHD-1X40" device=""/>
-<part name="U$2" library="auv" deviceset="ILLINOISAUV" device=""/>
 </parts>
 <sheets>
