File: jetson.sch (EAGLE design)
At the start: 5 parts, among them J101 80-PIN-CARD-EDGE

Commit message: Updates and fixes
Connections:
- net GND: no longer J101.P$38, J101.P$78
- net GPIO2: now also J101.P$35, J101.P$75; no longer J101.P$31, J101.P$71
- net GPIO3: now also J101.P$34, J101.P$74; no longer J101.P$30, J101.P$70
- net I2C_SCL: now also J101.P$37, J101.P$77; no longer J101.P$29, J101.P$69
- net I2C_SDA: now also J101.P$36, J101.P$76; no longer J101.P$28, J101.P$68
- net POWER_BUTTON: now also J101.P$27, J101.P$67; no longer J101.P$26, J101.P$66
- net RESET: no longer J101.P$27, J101.P$67
- net UART0_RX: now also J101.P$28, J101.P$68; no longer J101.P$37, J101.P$77
- net UART0_TX: now also J101.P$29, J101.P$69; no longer J101.P$36, J101.P$76
- net UART1_RX: now also J101.P$30, J101.P$70; no longer J101.P$35, J101.P$75
- net UART1_TX: now also J101.P$31, J101.P$71; no longer J101.P$34, J101.P$74
- net VIN: no longer J101.P$3, J101.P$4, J101.P$43, J101.P$44
