File: jetson.brd (EAGLE design)
At the start: 104.1 x 100 mm, 6 parts, among them J101 80-PIN-CARD-EDGE

Commit message: Updates and fixes
Parts:
- moved POWER 56.8 mm to (62.7, 20.3)
- moved U$2 52.5 mm to (28.6, 35.1), flipped to the bottom
- moved RESET 42.1 mm to (62.7, 29.5)
- moved U$1 36.7 mm to (49.5, 27.9), turned to 0 degrees
- moved RECOVERY 34.1 mm to (62.7, 38.4)
Connections:
- net GND: no longer J101.38, J101.78
- net GPIO2: now also J101.35, J101.75; no longer J101.31, J101.71
- net GPIO3: now also J101.34, J101.74; no longer J101.30, J101.70
- net I2C_SCL: now also J101.37, J101.77; no longer J101.29, J101.69
- net I2C_SDA: now also J101.36, J101.76; no longer J101.28, J101.68
- net POWER_BUTTON: now also J101.27, J101.67; no longer J101.26, J101.66
- net RESET: no longer J101.27, J101.67
- net UART0_RX: now also J101.28, J101.68; no longer J101.37, J101.77
- net UART0_TX: now also J101.29, J101.69; no longer J101.36, J101.76
- net UART1_RX: now also J101.30, J101.70; no longer J101.35, J101.75
- net UART1_TX: now also J101.31, J101.71; no longer J101.34, J101.74
- net VIN: no longer J101.3, J101.4, J101.43, J101.44
Routing:
- net VIN: track 120.1 -> 15.2 mm, vias 8 -> 4
- net RESET: track 84.3 -> 31.9 mm, vias 1 -> 0
- net UART0_TX: track 27.7 -> 63.3 mm
- net UART1_TX: track 27.2 -> 58.7 mm
- net POWER_BUTTON: track 98.0 -> 66.8 mm
- net UART0_RX: track 31.3 -> 62.4 mm
- net UART1_RX: track 30.3 -> 57.8 mm
- net GPIO0: track 27.2 -> 54.0 mm
- net GPIO2: track 28.2 -> 54.5 mm
- net GPIO1: track 30.8 -> 53.1 mm
- net I2C_SCL: track 29.3 -> 46.5 mm
- net GPIO3: track 31.8 -> 48.7 mm
- net I2C_SDA: track 32.9 -> 47.2 mm
- net RECOVERY: track 42.7 -> 34.5 mm
Other:
- board size 104.1 x 100 mm -> 104.1 x 53 mm
- board text added: "Orbitty Carrier"
- board text removed: "Orbitty Carrier Adrian Brandemuehl"
