File: speed_controllers.brd (EAGLE design)
At the start: 147.3 x 147.3 mm, 48 parts, among them M1 TE-1-1123723-3, M2 TE-1-1123723-3, M3 TE-1-1123723-3, M4 TE-1-1123723-3, M5 TE-1-1123723-3, M6 TE-1-1123723-3, M7 TE-1-1123723-3, M8 TE-1-1123723-3

Commit message: Add another hall effect and fix resistor value
Parts:
- added HE1: (no value), auv:1X03
- R10: value 10k -> 2k
Connections:
- net FET_G: now also HE1.3
- net GND: now also HE1.2
- net VCC: now also HE1.1
Routing:
- net FET_G: track 184.8 -> 202.1 mm
Changed lines of the file:
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@@
 <attribute name="SPICEPREFIX" value="C" x="-54.864" y="-12.192" size="1.778" layer="27" rot="R270" display="off"/>
 </element>
-<element name="R10" library="auv" package="R0603" value="10k" x="-62.992" y="-2.54"/>
+<element name="R10" library="auv" package="R0603" value="2k" x="-62.992" y="-2.54"/>
+<element name="HE1" library="auv" package="1X03" value="" x="1.016" y="-55.88"/>
 </elements>
 <signals>
@@
 <contactref element="R8" pad="2"/>
 <contactref element="R9" pad="2"/>
+<contactref element="HE1" pad="2"/>
 </signal>
 <signal name="VCC">
@@
 <contactref element="R10" pad="2"/>
 <contactref element="FET2" pad="S"/>
+<contactref element="HE1" pad="1"/>
 </signal>
 <signal name="FET_G">
@@
 <wire x1="27.305" y1="-40.005" x2="18.415" y2="-40.005" width="0.254" layer="16"/>
 <wire x1="18.415" y1="-40.005" x2="8.89" y2="-40.005" width="0.254" layer="16"/>
-<wire x1="8.89" y1="-40.005" x2="-4.445" y2="-40.005" width="0.254" layer="16"/>
+<wire x1="8.89" y1="-40.005" x2="0" y2="-40.005" width="0.254" layer="16"/>
+<wire x1="0" y1="-40.005" x2="-4.445" y2="-40.005" width="0.254" layer="16"/>
 <wire x1="-4.445" y1="-40.005" x2="-13.97" y2="-40.005" width="0.254" layer="16"/>
 <wire x1="-13.97" y1="-40.005" x2="-22.86" y2="-40.005" width="0.254" layer="16"/>
@@
 <wire x1="8.89" y1="-41.295" x2="8.89" y2="-40.005" width="0.254" layer="1"/>
 <wire x1="27.305" y1="-40.005" x2="36.83" y2="-40.005" width="0.254" layer="16"/>
+<contactref element="HE1" pad="3"/>
+<wire x1="0" y1="-52.07" x2="0" y2="-40.005" width="0.254" layer="16"/>
+<wire x1="3.556" y1="-55.88" x2="3.556" y2="-55.626" width="0.254" layer="16"/>
+<wire x1="3.556" y1="-55.626" x2="0" y2="-52.07" width="0.254" layer="16"/>
 </signal>
 <signal name="PWM_GND">

Commit message: Remove outer circle. Add logo
Parts:
- added U$2: (no value), auv:ILLINOISAUV
- moved U$1 15.8 mm to (14.1, 0.25)
Changed lines of the file:
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@@
 <text x="17.272" y="-10.414" size="1.27" layer="25" rot="R90">GND</text>
 <text x="25.654" y="-41.148" size="1.27" layer="26" rot="MR270">GND</text>
-<circle x="0" y="0" radius="127" width="0.254" layer="1"/>
 <text x="-12.065" y="52.07" size="1.778" layer="25" rot="R270">GND</text>
 <text x="-9.525" y="52.07" size="1.778" layer="25" rot="R270">GND</text>
@@
 <text x="12.7" y="58.42" size="1.778" layer="25" rot="R90">5V</text>
 <text x="10.16" y="58.42" size="1.778" layer="25" rot="R90">KILL</text>
-<text x="6.985" y="22.86" size="1.778" layer="22" rot="MR0">+</text>
-<text x="6.35" y="5.715" size="1.778" layer="22" rot="MR180">-</text>
+<text x="14.605" y="9.144" size="1.778" layer="22" rot="MR0">+</text>
+<text x="13.462" y="-8.001" size="1.778" layer="22" rot="MR180">-</text>
 <text x="-2.54" y="-10.16" size="1.27" layer="21" rot="R90">PWM</text>
 <text x="-15.24" y="-18.415" size="1.27" layer="21" rot="R90">PWM</text>
@@
 <element name="M7" library="auv" package="TE-1-1123723-3" value="TE-1-1123723-3" x="31.75" y="43.307" smashed="yes" rot="MR0"/>
 <element name="M8" library="auv" package="TE-1-1123723-3" value="TE-1-1123723-3" x="44.45" y="19.05" smashed="yes" rot="MR0"/>
-<element name="U$1" library="auv" package="XT-60" value="XT-60" x="6.731" y="14.224" rot="MR90"/>
+<element name="U$1" library="auv" package="XT-60" value="XT-60" x="14.097" y="0.254" rot="MR90"/>
 <element name="HE2" library="auv" package="1X03" value="" x="-54.483" y="-21.463" smashed="yes" rot="R90">
 <attribute name="NAME" x="-51.2318" y="-21.5392" size="1.27" layer="25" ratio="10" rot="R90"/>
@@
 <element name="R10" library="auv" package="R0603" value="2k" x="-62.992" y="-2.54"/>
 <element name="HE1" library="auv" package="1X03" value="" x="1.016" y="-55.88"/>
+<element name="U$2" library="auv" package="ILLINOISAUV" value="" x="0" y="0" rot="MR180"/>
 </elements>
 <signals>
