File: backplane.brd (EAGLE design)
At the start: 203.2 x 101.6 mm, 9 parts

Commit message: cleaning up for 2018
Parts:
- added BAT: XT-60, auv:XT-60
- added C1: 0.1uF, auv:C0603
- added DEPTH: DF13-4P-1.25DSA, auv:DF13-4P-1.25DSA
- added IC1: MAX3233ECPP, auv:DIL20
- added MODEM: (no value), auv:1X08
- PIXHAWK: value TE-2-5530843-0 -> PIXHAWK_EDGE_CONNCONN
- POWER: value TE-2-5530843-0 -> TE-5-5530843-0; device auv:TE-2-5530843-0 -> auv:TE-5-5530843-0
- moved POWER 49.1 mm to (31.0, 15.0)
- moved U$1 24.1 mm to (42.2, 77.2)
- moved PIXHAWK 9.40 mm to (70.6, 30.7)
- turned PWM to 270 degrees
Connections:
- removed net SPARTON_RX: U$3.UART0_TX
- removed net SPARTON_TX: U$3.UART0_RX
- new net +3V3: C1.1, IC1.9
- new net 5V: DEPTH.P$1
- new net MODEM_RS232_RX: IC1.7
- new net MODEM_RS232_TX: IC1.8
- new net MODEM_RX: IC1.4, U$3.UART0_TX
- new net MODEM_TX: IC1.6, U$3.UART0_RX
- new net PIXHAWK_GPIO3: PWM.17, U$3.GPIO3
- new net PIXHAWK_I2C_SCL: DEPTH.P$2, PIXHAWK.71, PIXHAWK.72
- new net PIXHAWK_I2C_SDA: DEPTH.P$3, PIXHAWK.73, PIXHAWK.74
- new net PWM1: PIXHAWK.39, PIXHAWK.40, PWM.1
- new net PWM2: PIXHAWK.41, PIXHAWK.42, PWM.3
- new net PWM3: PIXHAWK.43, PIXHAWK.44, PWM.5
- new net PWM4: PIXHAWK.45, PIXHAWK.46, PWM.7
- new net PWM5: PIXHAWK.47, PIXHAWK.48, PWM.9
- new net PWM6: PIXHAWK.49, PIXHAWK.50, PWM.11
- new net PWM7: PIXHAWK.51, PIXHAWK.52, PWM.13
- new net PWM8: PIXHAWK.53, PIXHAWK.54, PWM.15
- net +5V: now also PIXHAWK.1, PIXHAWK.2, PIXHAWK.3, PIXHAWK.4, PIXHAWK.5, PIXHAWK.6
- net GND: now also BAT.P$2, C1.2, DEPTH.P$4, IC1.18, PIXHAWK.75, PIXHAWK.76, PIXHAWK.77, PIXHAWK.78, PIXHAWK.79, PIXHAWK.80, PWM.10, PWM.12, PWM.14, PWM.16, PWM.18, PWM.2, PWM.20, PWM.4, PWM.6, PWM.8; no longer PWM.1, PWM.11, PWM.13, PWM.15, PWM.17, PWM.19, PWM.3, PWM.5, PWM.7, PWM.9
- net PIXHAWK_TELEM2_RX: now also PIXHAWK.10, PIXHAWK.9
- net PIXHAWK_TELEM2_TX: now also PIXHAWK.7, PIXHAWK.8
- net VBAT: now also BAT.P$1
Routing:
- net PIXHAWK_TELEM2_RX: track 0.00 -> 155.2 mm
- net PIXHAWK_TELEM2_TX: track 0.00 -> 153.4 mm
- net PWM1: track 0.00 -> 142.1 mm
- net PWM2: track 0.00 -> 138.6 mm
- net PWM3: track 0.00 -> 134.9 mm
- net PWM4: track 0.00 -> 131.3 mm
- net PWM5: track 0.00 -> 127.7 mm
- net PWM6: track 0.00 -> 124.2 mm
- net PWM7: track 0.00 -> 120.5 mm
- net PWM8: track 0.00 -> 116.9 mm
- net PIXHAWK_I2C_SDA: track 0.00 -> 110.1 mm, vias 0 -> 1
- net PIXHAWK_I2C_SCL: track 0.00 -> 108.1 mm
- net PIXHAWK_GPIO3: track 0.00 -> 62.5 mm
- net MODEM_TX: track 0.00 -> 59.5 mm
- net MODEM_RX: track 0.00 -> 55.9 mm
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- added copper zone on layer 1, net GND
- added copper zone on layer 16, net VBAT
- removed copper zone on layer 16, net GND
- removed copper zone on layer 1, net VBAT
