File: backplane.sch (EAGLE design)
At the start: 9 parts

Commit message: cleaning up for 2018
Parts:
- added BAT: XT-60, auv:XT-60
- added C1: 0.1uF, auv:C-EUC0603
- added DEPTH: DF13-4P-1.25DSA, auv:DF13-4P-1.25DSA
- added IC1: MAX3233ECPP, auv:MAX3233ECPP
- added MODEM: (no value), auv:PINHD-1X8
- PIXHAWK: value TE-2-5530843-0 -> PIXHAWK_EDGE_CONNCONN; device auv:TE-2-5530843-0 -> auv:PIXHAWK_EDGE_CONNCONN
- POWER: value TE-2-5530843-0 -> TE-5-5530843-0; device auv:TE-2-5530843-0 -> auv:TE-5-5530843-0
Connections:
- removed net SPARTON_RX: U$3.UART0_TX
- removed net SPARTON_TX: U$3.UART0_RX
- new net +3V3: C1.1, IC1P.VCC
- new net 5V: DEPTH.1
- new net MODEM_RS232_RX: IC1Q.T1OUT
- new net MODEM_RS232_TX: IC1Q.R1IN
- new net MODEM_RX: IC1Q.T1IN, U$3.UART0_TX
- new net MODEM_TX: IC1Q.R1OUT, U$3.UART0_RX
- new net PIXHAWK_GPIO3: PWM.17, U$3.GPIO3
- new net PIXHAWK_I2C_SCL: DEPTH.2, PIXHAWK.I2C_SCL
- new net PIXHAWK_I2C_SDA: DEPTH.3, PIXHAWK.I2C_SDA
- new net PWM1: PIXHAWK.PWM1, PWM.1
- new net PWM2: PIXHAWK.PWM2, PWM.3
- new net PWM3: PIXHAWK.PWM3, PWM.5
- new net PWM4: PIXHAWK.PWM4, PWM.7
- new net PWM5: PIXHAWK.PWM5, PWM.9
- new net PWM6: PIXHAWK.PWM6, PWM.11
- new net PWM7: PIXHAWK.PWM7, PWM.13
- new net PWM8: PIXHAWK.PWM8, PWM.15
- net +5V: now also PIXHAWK.5V
- net GND: now also BAT.2, C1.2, DEPTH.4, IC1P.GND, PIXHAWK.GND, PWM.10, PWM.12, PWM.14, PWM.16, PWM.18, PWM.2, PWM.20, PWM.4, PWM.6, PWM.8; no longer PWM.1, PWM.11, PWM.13, PWM.15, PWM.17, PWM.19, PWM.3, PWM.5, PWM.7, PWM.9
- net PIXHAWK_TELEM2_RX: now also PIXHAWK.TELEM2_RX
- net PIXHAWK_TELEM2_TX: now also PIXHAWK.TELEM2_TX
- net VBAT: now also BAT.1
Other:
- moved on the sheet: PWM
